File: pcb/starpet.kicad_pcb (KiCad board)
At the start: 2 copper layers, 105.4 x 82.1 mm, 7 parts, among them J1 Conn_01x04_Pin, J2 Conn_01x08_Pin, SW1 SW_Push, SW2 SW_Push, U1 DHT11, U2 XIAO-ESP32-C3-SMD

Commit message: feat: Made changes to firmware and customized board design
Parts:
- added G***: LOGO, LOGO, F.Cu at (178.5, 125.2)
- added G***: LOGO, LOGO, B.Cu at (153.6, 99.8)
- added G***: LOGO, LOGO, B.Cu at (177.6, 97.4)
Other:
- board text added: "Starpet!!!"
